File: Timer.sch (KiCad schematic (older format))
At the start: 11 parts

Commit message: Unknown timer changes
Parts:
- added 10k (x5), 10k?: R, symbol R
Connections:
- net GND: now also 10k?.1
- net VCC: now also 10k.1, 10k.1, 10k.1, 10k.1, 10k.1
- net at U?.10 (~{W}/~{RDYA}): now also P?.11 (P11)
- net at U?.11 (~{SYNCA}): now also P?.9 (P9), 10k.2
- net at U?.12 (RxDA): now also P?.1 (P1), 10k?.2
- net at U?.13 (~{RxCA}): now also P?.3 (P3), 10k.2
- net at U?.14 (~{TxCA}): now also P?.7 (P7), 10k.2
- net at U?.15 (TxDA): now also P?.5 (P5)
- net at U?.16 (~{DTRA}): now also P?.17 (P17)
- net at U?.17 (~{RTSA}): now also P?.13 (P13)
- net at U?.18 (~{CTSA}): now also P?.15 (P15), 10k.2
- net at U?.19 (~{DCDA}): now also P?.19 (P19), 10k.2
Other:
- moved on the sheet: P?
Changed lines of the file:
@@
 L CONN_02X10 P?
 U 1 1 58C07356
-P 5250 5350
-F 0 "P?" H 5250 5900 50  0000 C CNN
-F 1 "CONN_02X10" V 5250 5350 50  0000 C CNN
-F 2 "" H 5250 4150 50  0000 C CNN
-F 3 "" H 5250 4150 50  0000 C CNN
-	1    5250 5350
+P 6200 5350
+F 0 "P?" H 6200 5900 50  0000 C CNN
+F 1 "CONN_02X10" V 6200 5350 50  0000 C CNN
+F 2 "" H 6200 4150 50  0000 C CNN
+F 3 "" H 6200 4150 50  0000 C CNN
+	1    6200 5350
 	1    0    0    -1
 $EndComp
+$Comp
+L R 10k
+U 1 1 58C0765F
+P 4500 4550
+F 0 "10k" V 4580 4550 50  0000 C CNN
+F 1 "R" V 4500 4550 50  0000 C CNN
+F 2 "" V 4430 4550 50  0000 C CNN
+F 3 "" H 4500 4550 50  0000 C CNN
+	1    4500 4550
+	1    0    0    -1
+$EndComp
+$Comp
+L R 10k
+U 1 1 58C0777D
+P 4700 4550
+F 0 "10k" V 4780 4550 50  0000 C CNN
+F 1 "R" V 4700 4550 50  0000 C CNN
+F 2 "" V 4630 4550 50  0000 C CNN
+F 3 "" H 4700 4550 50  0000 C CNN
+	1    4700 4550
+	1    0    0    -1
+$EndComp
+$Comp
+L R 10k
+U 1 1 58C077CF
+P 4900 4550
+F 0 "10k" V 4980 4550 50  0000 C CNN
+F 1 "R" V 4900 4550 50  0000 C CNN
+F 2 "" V 4830 4550 50  0000 C CNN
+F 3 "" H 4900 4550 50  0000 C CNN
+	1    4900 4550
+	1    0    0    -1
+$EndComp
+$Comp
+L R 10k
+U 1 1 58C07810
+P 5100 4550
+F 0 "10k" V 5180 4550 50  0000 C CNN
+F 1 "R" V 5100 4550 50  0000 C CNN
+F 2 "" V 5030 4550 50  0000 C CNN
+F 3 "" H 5100 4550 50  0000 C CNN
+	1    5100 4550
+	1    0    0    -1
+$EndComp
+$Comp
+L R 10k
+U 1 1 58C0784F
+P 5300 4550
+F 0 "10k" V 5380 4550 50  0000 C CNN
+F 1 "R" V 5300 4550 50  0000 C CNN
+F 2 "" V 5230 4550 50  0000 C CNN
+F 3 "" H 5300 4550 50  0000 C CNN
+	1    5300 4550
+	1    0    0    -1
+$EndComp
+Connection ~ 4700 4400
+Connection ~ 4900 4400
+Connection ~ 5100 4400
+Connection ~ 4500 4400
+$Comp
+L VCC #PWR?
+U 1 1 58C07A3C
+P 5400 4400
+F 0 "#PWR?" H 5400 4250 50  0001 C CNN
+F 1 "VCC" H 5400 4550 50  0000 C CNN
+F 2 "" H 5400 4400 50  0000 C CNN
+F 3 "" H 5400 4400 50  0000 C CNN
+	1    5400 4400
+	1    0    0    -1
+$EndComp
+Wire Wire Line
+	4350 5000 5950 5000
+Wire Wire Line
+	4500 5000 4500 4700
+Wire Wire Line
+	4350 5200 5950 5200
+Wire Wire Line
+	4700 5200 4700 4700
+Wire Wire Line
+	4350 5300 5950 5300
+Wire Wire Line
+	4900 5300 4900 4700
+Wire Wire Line
+	4350 5700 5100 5700
+Wire Wire Line
+	5100 5700 5100 4700
+Wire Wire Line
+	4350 5900 5300 5900
+Wire Wire Line
+	5300 5900 5300 4700
+Wire Wire Line
+	4350 4900 5950 4900
+Connection ~ 4500 5000
+Wire Wire Line
+	4350 5100 5950 5100
+Connection ~ 4700 5200
+Connection ~ 4900 5300
+Wire Wire Line
+	4350 5400 5950 5400
+Wire Wire Line
+	4350 5600 5000 5600
+Wire Wire Line
+	5000 5600 5000 5500
+Wire Wire Line
+	5000 5500 5950 5500
+Wire Wire Line
+	5100 5600 5950 5600
+Connection ~ 5100 5600
+Wire Wire Line
+	4350 5800 5200 5800
+Wire Wire Line
+	5200 5800 5200 5700
+Wire Wire Line
+	5200 5700 5950 5700
+Wire Wire Line
+	5300 5800 5950 5800
+Connection ~ 5300 5800
+$Comp
+L R 10k?
+U 1 1 58C0819B
+P 5750 4550
+F 0 "10k?" V 5830 4550 50  0000 C CNN
+F 1 "R" V 5750 4550 50  0000 C CNN
+F 2 "" V 5680 4550 50  0000 C CNN
+F 3 "" H 5750 4550 50  0000 C CNN
+	1    5750 4550
+	1    0    0    -1
+$EndComp
+$Comp
+L GND #PWR?
+U 1 1 58C081FB
+P 5950 4400
+F 0 "#PWR?" H 5950 4150 50  0001 C CNN
+F 1 "GND" H 5950 4250 50  0000 C CNN
+F 2 "" H 5950 4400 50  0000 C CNN
+F 3 "" H 5950 4400 50  0000 C CNN
+	1    5950 4400
+	1    0    0    -1
+$EndComp
+Wire Wire Line
+	5750 4700 5750 4900
+Connection ~ 5750 4900
+Wire Wire Line
+	5750 4400 5950 4400
+Wire Wire Line
+	4500 4400 5400 4400
+Connection ~ 5300 4400
 $EndSCHEMATC
