File: z80.kicad_sch (KiCad schematic)
At the start: 21 parts, among them P1 CONN_01X04, P2 CONN_02X20, P3 CONN_01X10, U1 7400, U1001 Z8400, U1002 AT28C64B, U1003 AS6C1008, U1004 Z8420, U1005 74LS138, Y1 4MHz

Commit message: WIP solving ERC issues
Parts:
- added R101, R102, R103: 10k, symbol z80-rescue:R
- added unit 5 of U101
- P101: renamed from P1; symbol z80-rescue:CONN_01X04 -> Connector:Conn_01x04_Pin
- U101: renamed from U1; symbol z80-rescue:7400 -> 74xx:7400
- U106: renamed from U1004; footprint ~ -> DIP-40__600_ELL; symbol z80-rescue:Z8420 -> z80-ownSymbols:Z8420
- renumbered C1 to C101, C2 to C102, C3 to C103, C4 to C104, C5 to C105, C6 to C106, C7 to C107, C8 to C108, P2 to P102, P3 to P103, R1 to R104, R2 to R105, R3 to R106, U1001 to U102, U1002 to U103, U1003 to U104, U1005 to U105, Y1 to Y101
Connections:
- net +5V is gone; now on net VCC: P102.36 (P36)
- net ~{IOREQ} is gone; now on net ~{IORQ}: P102.16 (P16), U102.20 (~{IORQ})
- net CLK: now also P101.2 (Pin_2); no longer P101.3 (P3)
- net GND: now also P101.3 (Pin_3), U101.7 (GND); no longer P101.2 (P2), U101.7 (GND), U101.7 (GND), U101.7 (GND)
- net VCC: now also P101.4 (Pin_4), U106.26 (VCC), R101.1, R102.1, R103.1, U101.14 (VCC); no longer P101.1 (P1), U101.14 (VCC), U101.14 (VCC), U101.14 (VCC), U102.17 (~{NMI}), U102.24 (~{WAIT}), U102.25 (~{BUSREQ}), U106.28 (B1)
- net ~{BUSACK}: now also U102.23 (~{BUSACK})
- net ~{BUSREQ}: now also U102.25 (~{BUSREQ}), R102.2
- net ~{RESET}: now also P101.1 (Pin_1); no longer P101.4 (P4)
- net ~{WAIT}: now also U102.24 (~{WAIT}), R103.2
- net ~{CE_1} renamed ~{CTC_CE}
- net ~{CTC_CE}: now also P102.40 (P40); no longer P102.38 (P38)
- net ~{CE_2} renamed ~{SIO_CE}
- net ~{SIO_CE}: now also P102.38 (P38); no longer P102.40 (P40)
- new net ~{NMI}: R101.2, U102.17 (~{NMI})
- no-connect marks 18 -> 17
Other:
- moved on the sheet: C101, C102, C103, C104, C105, C106

Commit message: Fixed all schematic ERC errors and warnings
Parts:
- added unit 4 of U101
- C101, C102, C103, C104, C105, C106, C107, C108: symbol z80-rescue:C -> Device:C
- P102: symbol z80-rescue:CONN_02X20 -> Connector_Generic:Conn_02x20_Odd_Even
- P103: symbol z80-rescue:CONN_01X10 -> Connector:Conn_01x10_Pin
- R101, R102, R103, R104, R105, R106: symbol z80-rescue:R -> Device:R
- U102: footprint (none) -> Package_DIP:DIP-40_W15.24mm_Socket_LongPads; symbol z80-rescue:Z8400 -> z80-ownSymbols:Z8400
- U103: symbol z80-rescue:AT28C64B -> z80-ownSymbols:AT28C64B
- U104: footprint ~ -> Package_DIP:DIP-32_W15.24mm_LongPads; symbol z80-rescue:AS6C1008 -> z80-ownSymbols:AS6C1008
- U105: footprint ~ -> Package_DIP:DIP-16_W7.62mm_Socket_LongPads; symbol z80-rescue:74LS138 -> 74xx:74LS138
- U106: footprint DIP-40__600_ELL -> Package_DIP:DIP-40_W15.24mm_LongPads
- Y101: symbol z80-rescue:Crystal -> Device:Crystal
Connections:
- net A0: now also P102.18 (Pin_18); no longer P102.17 (P17)
- net A1: now also P102.20 (Pin_20); no longer P102.19 (P19)
- net A10: now also P102.38 (Pin_38); no longer P102.37 (P37)
- net A11: now also P102.40 (Pin_40); no longer P102.39 (P39)
- net A12: now also P102.1 (Pin_1); no longer P102.2 (P2)
- net A13: now also P102.3 (Pin_3); no longer P102.4 (P4)
- net A14: now also P102.5 (Pin_5); no longer P102.6 (P6)
- net A15: now also P102.7 (Pin_7); no longer P102.8 (P8)
- net A2: now also P102.22 (Pin_22); no longer P102.21 (P21)
- net A3: now also P102.24 (Pin_24); no longer P102.23 (P23)
- net A4: now also P102.26 (Pin_26); no longer P102.25 (P25)
- net A5: now also P102.28 (Pin_28); no longer P102.27 (P27)
- net A6: now also P102.30 (Pin_30); no longer P102.29 (P29)
- net A7: now also P102.32 (Pin_32); no longer P102.31 (P31)
- net A8: now also P102.34 (Pin_34); no longer P102.33 (P33)
- net A9: now also P102.36 (Pin_36); no longer P102.35 (P35)
- net CLK: now also P102.25 (Pin_25); no longer P102.26 (P26)
- net D0: now also P102.2 (Pin_2); no longer P102.1 (P1)
- net D1: now also P102.4 (Pin_4); no longer P102.3 (P3)
- net D2: now also P102.6 (Pin_6); no longer P102.5 (P5)
- net D3: now also P102.8 (Pin_8); no longer P102.7 (P7)
- net D4: now also P102.10 (Pin_10); no longer P102.9 (P9)
- net D5: now also P102.12 (Pin_12); no longer P102.11 (P11)
- net D6: now also P102.14 (Pin_14); no longer P102.13 (P13)
- net D7: now also P102.16 (Pin_16); no longer P102.15 (P15)
- net GND: now also P102.9 (Pin_9), U101.12, U101.13; no longer P102.10 (P10), P102.34 (P34)
- net VCC: now also P102.33 (Pin_33); no longer P102.36 (P36)
- net ~{BUSACK}: now also P102.31 (Pin_31); no longer P102.32 (P32)
- net ~{BUSREQ}: now also P102.29 (Pin_29); no longer P102.30 (P30)
- net ~{CTC_CE}: now also P102.35 (Pin_35); no longer P102.40 (P40)
- net ~{INT}: now also P102.23 (Pin_23); no longer P102.24 (P24)
- net ~{IORQ}: now also P102.15 (Pin_15); no longer P102.16 (P16)
- net ~{M1}: now also P102.11 (Pin_11); no longer P102.12 (P12)
- net ~{MREQ}: now also P102.13 (Pin_13); no longer P102.14 (P14)
- net ~{RD}: now also P102.17 (Pin_17); no longer P102.18 (P18)
- net ~{RESET}: now also P102.27 (Pin_27); no longer P102.28 (P28)
- net ~{SIO_CE}: now also P102.37 (Pin_37); no longer P102.38 (P38)
- net ~{WAIT}: now also P102.21 (Pin_21); no longer P102.22 (P22)
- net ~{WR}: now also P102.19 (Pin_19); no longer P102.20 (P20)
- net ~{CE_3}: now reaches U105.12 (O3)
- net ~{CE_3}: now also P102.39 (Pin_39)
Other:
- moved on the sheet: U103
