File: z80.kicad_pcb (KiCad board)
At the start: 2 copper layers, 60 parts, among them J201 Conn_02x06_Row_Letter_First, P101 CONN_01X04, P102 CONN_02X20, P103 CONN_01X10, P104 CONN_01X10, P105 CONN_02X20, P201 Interrupt Daisy Chain SIO, P202 Interrupt Daisy Chain CTC, P203 CONN_02X10, P204 Outputs, P205 Inputs, U101 7400, U102 Z8400, U103 AT28C64B, U104 AS6C1008, U105 74LS138, U106 Z8420, U201 Z8430, U202 Z8440, Y101 4MHz

Commit message: PCB routing almost complete
Parts:
- C201, C202: moved to B.Cu
- J201: footprint Connector_PinHeader_2.54mm:PinHeader_2x06_P2.54mm_Vertical -> Connector_PinHeader_2.54mm:PinHeader_2x06_P2.54mm_Horizontal
- P201, P202: footprint Connector_PinHeader_2.54mm:PinHeader_1x04_P2.54mm_Vertical -> Connector_PinHeader_2.54mm:PinHeader_1x03_P2.54mm_Vertical
- R201: renamed from 10k201; value R -> 10k; moved to B.Cu
- R202: renamed from 10k202; value R -> 10k; moved to B.Cu
- R203: renamed from 10k203; value R -> 10k; moved to B.Cu
- R204: renamed from 10k204; value R -> 10k; moved to B.Cu
- R205: renamed from 10k206; value R -> 10k; moved to B.Cu
- R206: renamed from 10k205; value R -> 10k; moved to B.Cu
- R207: renamed from 10k207; value R -> 10k; moved to B.Cu
- R208: renamed from 10k208; value R -> 10k; moved to B.Cu
- R209: renamed from 10k209; value R -> 10k; moved to B.Cu
- R210: renamed from 10k210; value R -> 10k; moved to B.Cu
- R211: renamed from 10k211; value R -> 10k; moved to B.Cu
- R212: renamed from 10k212; value R -> 10k; moved to B.Cu
- R213: renamed from 10k213; value R -> 10k; moved to B.Cu
- R214: renamed from 10k214; value R -> 10k; moved to B.Cu
- R215: renamed from 10k215; value R -> 10k; moved to B.Cu
- R216: renamed from R201; moved to B.Cu
- R217: renamed from R202; moved to B.Cu
- moved R210 93.7 mm to (205.1, 210.6), turned to -90 degrees
- moved R208 69.5 mm to (207.6, 210.6), turned to -90 degrees
- moved R207 66.4 mm to (210.2, 210.6), turned to -90 degrees
- moved R216 47.5 mm to (235.6, 222.6), turned to -90 degrees
- moved R217 47.3 mm to (235.6, 227.3), turned to -90 degrees
- moved R203 42.6 mm to (245.1, 223.5), turned to 90 degrees
- moved R205 38.4 mm to (249.6, 223.5), turned to 90 degrees
- moved R204 33.7 mm to (254.0, 223.5), turned to 90 degrees
- moved R202 30.0 mm to (258.2, 223.5), turned to 90 degrees
- moved R201 26.5 mm to (262.6, 223.5), turned to 90 degrees
- moved R209 26.5 mm to (266.1, 223.5), turned to 90 degrees
- moved J201 13.0 mm to (231.1, 228.6), turned to -90 degrees
- moved R214 11.9 mm to (283.6, 210.8), turned to 180 degrees
- moved R215 10.7 mm to (283.6, 213.4), turned to 180 degrees
- moved R212 10.1 mm to (283.6, 200.7), turned to 180 degrees
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- renumbered R203 to R218
Connections:
- net Net-(P201-Pin_3) renamed /Timer/IEO_SIO
- J201 pad 1: (no net) -> unconnected-(J201-Pin_1-Pad1)
- J201 pad 10: (no net) -> /Timer/TxDB3.3V
- J201 pad 11: (no net) -> unconnected-(J201-Pin_11-Pad11)
- J201 pad 12: (no net) -> /Timer/~{RTSB}
- J201 pad 2: (no net) -> GND
- J201 pad 3: (no net) -> unconnected-(J201-Pin_3-Pad3)
- J201 pad 4: (no net) -> /Timer/~{CTSB}
- J201 pad 5: (no net) -> unconnected-(J201-Pin_5-Pad5)
- J201 pad 6: (no net) -> VCC
- J201 pad 7: (no net) -> unconnected-(J201-Pin_7-Pad7)
- J201 pad 8: (no net) -> /Timer/RxDB
- J201 pad 9: (no net) -> unconnected-(J201-Pin_9-Pad9)
- P105 pad 1: A12 -> unconnected-(P105-Pin_1-Pad1)
- P105 pad 13: ~{MREQ} -> unconnected-(P105-Pin_13-Pad13)
- P105 pad 19: ~{WR} -> unconnected-(P105-Pin_19-Pad19)
- P105 pad 21: ~{WAIT} -> unconnected-(P105-Pin_21-Pad21)
- P105 pad 22: A2 -> unconnected-(P105-Pin_22-Pad22)
- P105 pad 24: A3 -> unconnected-(P105-Pin_24-Pad24)
- P105 pad 26: A4 -> unconnected-(P105-Pin_26-Pad26)
- P105 pad 28: A5 -> unconnected-(P105-Pin_28-Pad28)
- P105 pad 29: ~{BUSREQ} -> unconnected-(P105-Pin_29-Pad29)
- P105 pad 3: A13 -> unconnected-(P105-Pin_3-Pad3)
- P105 pad 30: A6 -> unconnected-(P105-Pin_30-Pad30)
- P105 pad 31: ~{BUSACK} -> unconnected-(P105-Pin_31-Pad31)
- P105 pad 32: A7 -> unconnected-(P105-Pin_32-Pad32)
- P105 pad 34: A8 -> unconnected-(P105-Pin_34-Pad34)
- P105 pad 36: A9 -> unconnected-(P105-Pin_36-Pad36)
- P105 pad 38: A10 -> unconnected-(P105-Pin_38-Pad38)
- P105 pad 39: ~{CE_3} -> unconnected-(P105-Pin_39-Pad39)
- P105 pad 40: A11 -> unconnected-(P105-Pin_40-Pad40)
- P105 pad 5: A14 -> unconnected-(P105-Pin_5-Pad5)
- P105 pad 7: A15 -> unconnected-(P105-Pin_7-Pad7)
- P201 pad 2: Net-(P201-Pin_2) -> /Timer/IEI_SIO
- P202 pad 2: ~{INT} -> /Timer/IEI_CTC
- R216 pad 2: Net-(J201-Pin_b5) -> /Timer/TxDB3.3V
- R217 pad 1: Net-(J201-Pin_b5) -> /Timer/TxDB3.3V
- U202 pad 5: Net-(P201-Pin_2) -> ~{INT}
- U202 pad 6: Net-(P201-Pin_4) -> /Timer/IEI_SIO
Routing:
- net VCC: track 432.9 -> 681.8 mm, vias 13 -> 19
- net GND: track 438.1 -> 685.2 mm, vias 15 -> 22
- net CLK: track 100.7 -> 281.8 mm, vias 4 -> 6
- net /Timer/RxDB: track 0.00 -> 104.0 mm, vias 0 -> 2
- net /Timer/~{RTSB}: track 0.00 -> 97.3 mm, vias 0 -> 2
- net ~{RD}: track 178.5 -> 274.7 mm, vias 6 -> 10
- net ~{RESET}: track 154.5 -> 243.9 mm, vias 3 -> 5
- net D0: track 177.6 -> 258.7 mm, vias 8 -> 11
- net /Timer/IEI_CTC: track 0.00 -> 80.5 mm, vias 0 -> 2
- net /Timer/~{CTSB}: track 0.00 -> 79.6 mm, vias 0 -> 2
- net ~{IORQ}: track 104.1 -> 183.7 mm, vias 3 -> 5
- net ~{M1}: track 86.1 -> 161.3 mm, vias 2 -> 4
- net D2: track 172.5 -> 247.4 mm, vias 4 -> 7
- net /Timer/IEO_CTC: track 0.00 -> 72.9 mm, vias 0 -> 2
- net ~{INT}: track 133.6 -> 204.6 mm, vias 4 -> 6
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Other:
- board text added: "0"
- board text added: "1"
- board text added: "2"
- board text added: "3"
- board text added: "BLACK"
- board text added: "CLK/TRG"
- board text added: "CTC"
- board text added: "FTDI USB-Serial SIO B"
- board text added: "GREEN"
- board text added: "IEO"
- board text added: "NC"
- board text added: "RxDA"
- board text added: "RxDB"
- board text added: "SIO"
- board text added: "TxDA"
- board text added: "TxDB"
- board text added: "ZC/TO"
- board text added: "~{CTSA}"
- board text added: "~{CTSB}"
- board text added: "~{DCDA}"
- board text added: "~{DCDB}"
- board text added: "~{DTRA}"
- board text added: "~{DTRB}"
- board text added: "~{RTSA}"
- board text added: "~{RTSB}"
- board text added: "~{RxCA}"
- board text added: "~{RxTxCB}"
- board text added: "~{SYNCA}"
- board text added: "~{SYNCB}"
- board text added: "~{TxCA}"
- board text added: "~{W}/~{RDYA}"
- board text added: "~{W}/~{RDYB}"
- board text removed: "CLK/TRG0"
- board text removed: "CLK/TRG1"
- board text removed: "CLK/TRG2"
- board text removed: "CLK/TRG3"
- board text removed: "ZC/TO0"
- board text removed: "ZC/TO1"
- board text removed: "ZC/TO2"

Commit message: Removed serial board which has now been moved to its own project.
Parts:
- removed C201, C202: 0.1u, Capacitor_SMD:C_0805_2012Metric_Pad1.18x1.45mm_HandSolder
- removed C203: 10u, Capacitor_THT:CP_Radial_D10.0mm_P5.00mm
- removed D201: LED, LED_SMD:LED_0805_2012Metric_Pad1.15x1.40mm_HandSolder
- removed J201: Conn_02x06_Row_Letter_First, Connector_PinHeader_2.54mm:PinHeader_2x06_P2.54mm_Horizontal
- removed P201: Interrupt Daisy Chain SIO, Connector_PinHeader_2.54mm:PinHeader_1x03_P2.54mm_Vertical
- removed P202: Interrupt Daisy Chain CTC, Connector_PinHeader_2.54mm:PinHeader_1x03_P2.54mm_Vertical
- removed P203: CONN_02X10, Connector_PinHeader_2.54mm:PinHeader_2x10_P2.54mm_Vertical
- removed P204: Outputs, Connector_PinHeader_2.54mm:PinHeader_1x03_P2.54mm_Vertical
- removed P205: Inputs, Connector_PinHeader_2.54mm:PinHeader_1x04_P2.54mm_Vertical
- removed R201, R202, R203, R204, R205, R206, R207, R208, R209, R210, R211, R212, R213, R214, R215, R216: 10k, Resistor_SMD:R_0805_2012Metric_Pad1.20x1.40mm_HandSolder
- removed R217: 15k, Resistor_SMD:R_0805_2012Metric_Pad1.20x1.40mm_HandSolder
- removed R218: 470, Resistor_SMD:R_0805_2012Metric_Pad1.20x1.40mm_HandSolder
- removed U201: Z8430, Package_DIP:DIP-28_W15.24mm_Socket
- removed U202: Z8440, Package_DIP:DIP-40_W15.24mm_Socket_LongPads
- P105: value CONN_02X20 -> ~; footprint Connector_PinHeader_2.54mm:PinHeader_2x20_P2.54mm_Horizontal -> Connector_PinHeader_2.54mm:PinHeader_1x03_P2.54mm_Vertical
- moved P105 95.9 mm to (149.9, 228.0), turned to 0 degrees
Connections:
- P105 pad 1: unconnected-(P105-Pin_1-Pad1) -> /PIO_IEO
- P105 pad 2: D0 -> /PIO_IEI
- P105 pad 3: unconnected-(P105-Pin_3-Pad3) -> VCC
- U106 pad 22: unconnected-(U106-IEO-Pad22) -> /PIO_IEO
- U106 pad 24: GND -> /PIO_IEI
Routing:
- net GND: track 685.2 -> 434.3 mm, vias 22 -> 15
- net VCC: track 681.8 -> 445.0 mm, vias 19 -> 13
- net /Timer/RxDB: track 104.0 -> 0.00 mm, vias 2 -> 0
- net /Timer/~{RTSB}: track 97.3 -> 0.00 mm, vias 2 -> 0
- net ~{RD}: track 274.7 -> 178.5 mm, vias 10 -> 6
- net ~{RESET}: track 243.9 -> 154.5 mm, vias 5 -> 3
- net D0: track 258.7 -> 177.6 mm, vias 11 -> 8
- net /Timer/IEI_CTC: track 80.5 -> 0.00 mm, vias 2 -> 0
- net /Timer/~{CTSB}: track 79.6 -> 0.00 mm, vias 2 -> 0
- net ~{M1}: track 161.3 -> 86.1 mm, vias 4 -> 2
- net D2: track 247.4 -> 172.5 mm, vias 7 -> 4
- net CLK: track 281.8 -> 207.6 mm, vias 6 -> 5
- net /Timer/IEO_CTC: track 72.9 -> 0.00 mm, vias 2 -> 0
- net A0: track 199.4 -> 129.1 mm, vias 7 -> 5
- net D1: track 248.0 -> 178.4 mm, vias 9 -> 7
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Other:
- board outline added: 123.8 x 87 mm
- board text added: "39"
- board text added: "40"
- board text added: "A0"
- board text added: "A7"
- board text added: "ARDY"
- board text added: "B0"
- board text added: "B7"
- board text added: "BRDY"
- board text added: "PIO IEI"
- board text added: "PIO IEO"
- board text added: "~{ASTB}"
- board text added: "~{BSTB}"
- board text removed: "0"
- board text removed: "3"
- board text removed: "BLACK"
- board text removed: "CLK/TRG"
- board text removed: "CTC"
- board text removed: "FTDI USB-Serial SIO B"
- board text removed: "GREEN"
- board text removed: "IEO"
- board text removed: "NC"
- board text removed: "RxDA"
- board text removed: "RxDB"
- board text removed: "SIO"
- board text removed: "TxDA"
- board text removed: "TxDB"
- board text removed: "ZC/TO"
- board text removed: "~{CTSA}"
- board text removed: "~{CTSB}"
- board text removed: "~{DCDA}"
- board text removed: "~{DCDB}"
- board text removed: "~{DTRA}"
- board text removed: "~{DTRB}"
- board text removed: "~{RTSA}"
- board text removed: "~{RTSB}"
- board text removed: "~{RxCA}"
- board text removed: "~{RxTxCB}"
- board text removed: "~{SYNCA}"
- board text removed: "~{SYNCB}"
- board text removed: "~{TxCA}"
- board text removed: "~{W}/~{RDYA}"
- board text removed: "~{W}/~{RDYB}"

Commit message: Completed and ordered.
Other:
- board text added: "Z80 CPU Card v1.0 2025-12-01"
Changed lines of the file:
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@@
 		(grid_origin 25.4 152.4)
 		(pcbplotparams
-			(layerselection 0x00000000_00000000_00000000_000000a5)
+			(layerselection 0x00000000_00000000_55555555_5755f5ff)
 			(plot_on_all_layers_selection 0x00000000_00000000_00000000_00000000)
 			(disableapertmacros no)
@@
 			(subtractmaskfromsilk no)
 			(outputformat 1)
-			(mirror yes)
-			(drillshape 2)
+			(mirror no)
+			(drillshape 0)
 			(scaleselection 1)
-			(outputdirectory "/Users/andreas/Desktop/")
+			(outputdirectory "fabrication/")
 		)
 	)
@@
 		(layer "F.SilkS")
 		(effects
+			(font
+				(size 1 1)
+				(thickness 0.15)
+			)
+			(justify left bottom)
+		)
+	)
+	(gr_text "Z80 CPU Card v1.0 2025-12-01"
+		(at 29.845 234.315 0)
+		(layer "F.SilkS")
+		(effects
